File: SimpleCANBreakoutMicro.kicad_sch (KiCad schematic)
At the start: 12 parts, among them J1 Conn_01x04_Pin, J2 Conn_01x04_Pin, U2 XC6206PxxxMR, U3 SN65HVD230

Commit message: Add bottom pads, silkscreen
Parts:
- added TP1, TP2, TP3, TP4: TestPoint, TestPoint:TestPoint_Pad_1.0x1.0mm, symbol Connector:TestPoint
Connections:
- net +5V: now also TP1.1
- net CANH: now also TP2.1
- net CANL: now also TP3.1
- net GND: now also TP4.1

Commit message: Add Schematic
Other:
- note added: "3V3"
- note added: "CAN"
- note added: "CAN Connection"
- note added: "JST-GH & Test Points"
- note added: "MCU Connection"
- moved on the sheet: C1, C2, C3, C4, C5, C6, J1, J2, JP1, R1, TP1, TP2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

Commit message: Schematic title block (title, date, rev 1.0); PDF re-exported
Other:
- title: (none) -> SimpleCANBreakoutMicro
Changed lines of the file:
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@@
 	(generator_version "10.0")
 	(paper "A4")
+	(title_block
+		(title "SimpleCANBreakoutMicro")
+		(date "2026-10-17")
+		(rev "1.0")
+	)
 	(rectangle
 		(start 113.03 12.7)
